File: Eagle PCB files/TPS61165.sch (EAGLE design)
At the start: 50 parts, among them IC1 555, J1 DC-005, U1 TPS61165DBVRDBV0006A_L, U2 TPS61165DBVRDBV0006A_L

Commit message: Updated PCB files
Parts:
- removed D10, D11, D15, D16, D17, D18, D19, D20, D21, D22, D23, D24, D5, D6, D7, D8, D9: MP3030_N, MP3030:MP3030_N
- removed D12: 40V-500MA, OPL_Discrete_Semiconductor:SMD-DIODE-SCHOTTKY-40V-500MA(SOD-123)
- removed D13, D14: 20V-500MA, OPL_Discrete_Semiconductor:SMD-DIODE-SCHOTTKY-20V-500MA(SOD-123)
- removed R4, R5: 0R, Resistor:R_CHIP-0603(1608-METRIC)
- removed R6, R7: 0R, Resistor:R_CHIP-1206(3216-METRIC)
- added CTRL, TRIG: TPB1,27, testpad:TPB1,27
- added J2: (no value), SparkFun-Connectors:USB_MICRO-B_SMT
- added JP1: PINHD-2X4, Connector:PINHD-2X4
- D2: value MP3030_N -> 40V-500MA; device MP3030:MP3030_N -> OPL_Discrete_Semiconductor:SMD-DIODE-SCHOTTKY-40V-500MA(SOD-123)
- D3, D4: value MP3030_N -> 20V-500MA; device MP3030:MP3030_N -> OPL_Discrete_Semiconductor:SMD-DIODE-SCHOTTKY-20V-500MA(SOD-123)
- J1: value DC-005 -> (none); device OPL_Connector:CONN-POWER-JACK-2.1MM(DC-005) -> Connector:694108106102
- R1, R2: value 0.5Ω -> 1R
- VR1: value 10k -> 100k; device SparkFun-Resistors:POTENTIOMETER-PTH-9MM-1/20W-20% -> MP3030:5PIN-POT
Connections:
- removed net 12V: C1.1, C4.1, IC1./RES, IC1.VCC+, J1.+, L1.1, L2.1, R3.2, U1.VIN, U2.VIN
- removed net N$1: D17.2, D18.1
- removed net N$11: D10.2, D11.1
- removed net N$12: IC1.OUT, R5.1
- removed net N$13: D15.2, D16.1
- removed net N$15: D16.2, D17.1
- removed net N$17: D18.2, D19.1
- removed net N$18: D23.2, D24.1
- removed net N$19: D22.2, D23.1
- removed net N$2: D2.2, D3.1
- removed net N$20: D21.2, D22.1
- removed net N$21: D20.2, D21.1
- removed net N$3: D7.2, D8.1
- removed net N$4: D3.2, D4.1
- removed net N$5: D8.2, D9.1
- removed net N$6: D4.2, D5.1
- removed net N$7: D10.1, D9.2
- removed net N$8: D5.2, D6.1
- new net VCC: C1.1, C4.1, IC1./RES, IC1.VCC+, J1.1, J2.VBUS, L1.1, L2.1, R3.2, U1.VIN, U2.VIN
- net CTRL: now also CTRL.TP, IC1.OUT; no longer R5.2
- net DISCHARGE: now also D3.+, D4.-; no longer D13.+, D14.-
- net GND: now also J1.2, J1.3, J2.GND; no longer J1.-, R6.1, R6.2, R7.1, R7.2
- net LED1_N: now also JP1.6, JP1.8; no longer D11.2, D6.2
- net LED1_P: now also JP1.2, JP1.4; no longer D2.1, D7.1
- net LED2_N: now also JP1.5, JP1.7; no longer D19.2, D24.2
- net LED2_P: now also D2.-, JP1.1, JP1.3; no longer D12.-, D15.1, D20.1
- net N$10: now also D4.+, VR1.P$1; no longer D14.+, VR1.E
- net N$9: now also D3.-, VR1.P$3; no longer D13.-, VR1.A
- net SW1: now also D2.+; no longer D12.+
- net TRIGGER: now also TRIG.TP, VR1.P$2; no longer R4.1, R4.2, VR1.S
Other:
- note added: "3V *12 = 36V 65mA (typ.) to 200mA (max)"
- note added: "96 LED/ 48 per channel 1 channel: 3V*12 in series * 4 parallel group Voltage: 36V Current: Min: 65mA*4 = 260mA Max: 150mA*4 = 600mA"
- note added: "Driver 1"
- note added: "Driver 2"
- note added: "Holes"
- note added: "LED"
- note added: "MP3030-110H: 3V 65mA"
- note added: "PWM"
- note added: "Power Input"
- note added: "Rset: Min: 4*65mA=200mV/R R=0.769 Max: 4*150mA=200mV/R R=0.333"
- note removed: "12.2V"
- note removed: "18.2V"
- note removed: "2*200mA=200mV/0.5R"
- note removed: "200mV"
- note removed: "24.2V"
- note removed: "30.2V"
- note removed: "6.2V"
- note removed: "6V *5 = 30V 150mA (typ.) to 200mA (max)"
- note removed: "MP3030-1100: 3V 150mA"
- moved on the sheet: C1, C2, C3, C4, C5, C6, C7, C8, D1, H1, H2, H3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
